File: PWM-PCA9685.kicad_pcb (KiCad board)
At the start: 2 copper layers, 158.5 x 103.5 mm, 121 parts, among them J1 Conn_02x16_Top_Bottom, J2 Conn_02x16_Top_Bottom, J3 Conn_02x16_Top_Bottom, J4 Conn_02x20_Odd_Even, J5 Conn_02x12_Top_Bottom, Q1 SQJB00EP-T1_GE3, Q10 SQJB00EP-T1_GE3, Q11 SQJB00EP-T1_GE3, Q12 SQJB00EP-T1_GE3, Q13 SQJB00EP-T1_GE3, Q14 SQJB00EP-T1_GE3, Q15 SQJB00EP-T1_GE3, Q16 SQJB00EP-T1_GE3, Q17 SQJB00EP-T1_GE3, Q18 SQJB00EP-T1_GE3, Q19 SQJB00EP-T1_GE3, Q2 SQJB00EP-T1_GE3, Q20 SQJB00EP-T1_GE3, Q21 SQJB00EP-T1_GE3, Q22 SQJB00EP-T1_GE3, Q23 SQJB00EP-T1_GE3, Q24 SQJB00EP-T1_GE3, Q3 SQJB00EP-T1_GE3, Q4 SQJB00EP-T1_GE3, Q5 SQJB00EP-T1_GE3, Q6 SQJB00EP-T1_GE3, Q7 SQJB00EP-T1_GE3, Q8 SQJB00EP-T1_GE3, Q9 SQJB00EP-T1_GE3, U1 PCA9685PW, U2 PCA9685PW, U3 PCA9685PW

Commit message: updated
Parts:
- added C1: 47uF, Capacitor_THT:CP_Radial_D6.3mm_P2.50mm, F.Cu at (115.0, 100.0)
- added C2: 47uF, Capacitor_THT:CP_Radial_D6.3mm_P2.50mm, F.Cu at (125.0, 100.0)
- added C3: 47uF, Capacitor_THT:CP_Radial_D6.3mm_P2.50mm, F.Cu at (36.0, 39.5)
- added C4: 47uF, Capacitor_THT:CP_Radial_D6.3mm_P2.50mm, F.Cu at (46.0, 39.5)
- added D49: LED, LED_SMD:LED_0603_1608Metric, F.Cu at (146.0, 43.0)
- added D50: LED, LED_SMD:LED_0603_1608Metric, F.Cu at (150.0, 43.0)
- added R21: 1K, Resistor_SMD:R_0603_1608Metric, F.Cu at (146.0, 47.0)
- added R22: 1K, Resistor_SMD:R_0603_1608Metric, F.Cu at (150.0, 47.0)
- C5: renamed from C1; footprint Capacitor_SMD:C_0603_1608Metric -> Capacitor_SMD:C_1206_3216Metric
- C6: renamed from C2; footprint Capacitor_SMD:C_0603_1608Metric -> Capacitor_SMD:C_1206_3216Metric
- C7: renamed from C3; footprint Capacitor_SMD:C_0603_1608Metric -> Capacitor_SMD:C_1206_3216Metric
- moved C7 1.71 mm to (139.2, 71.0)
- moved C5 1.71 mm to (59.2, 71.0)
- moved C6 1.71 mm to (99.2, 71.0)
- moved D1 1.00 mm to (37.0, 90.5)
- moved D10 1.00 mm to (37.0, 67.7)
- moved D11 1.00 mm to (47.0, 70.2)
- moved D12 1.00 mm to (47.0, 67.7)
- moved D13 1.00 mm to (47.0, 55.0)
- moved D14 1.00 mm to (47.0, 52.5)
- moved D15 1.00 mm to (37.0, 54.9)
- moved D16 1.00 mm to (37.0, 52.6)
- moved D17 1.00 mm to (77.0, 90.5)
- moved D18 1.00 mm to (77.0, 88.0)
- moved D19 1.00 mm to (87.0, 90.5)
- moved D2 1.00 mm to (37.0, 88.0)
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Connections:
- J4 pad 40: Net-(J4-Pad40) -> ~OE
- U1 pad 23: GND -> ~OE
- U2 pad 23: GND -> ~OE
- U3 pad 23: GND -> ~OE
Routing:
- net ~OE: track 0.00 -> 209.9 mm, vias 0 -> 10
- net +12V: track 571.2 -> 610.5 mm, vias 0 -> 1
- net +5V: track 257.8 -> 295.1 mm
- net /A25: track 46.8 -> 58.3 mm
- net /A35: track 46.8 -> 58.2 mm
- net /A15: track 47.3 -> 58.4 mm
- net GND: track 68.8 -> 75.8 mm, vias 117 -> 184
- net SDA: track 203.0 -> 206.1 mm
- net SCL: track 206.9 -> 209.9 mm
- net Net-(D50-Pad2): track 0.00 -> 2.42 mm
- net Net-(D49-Pad2): track 0.00 -> 2.42 mm
- net PWM15: track 40.0 -> 38.8 mm
- net PWM14: track 38.0 -> 37.0 mm
- net PWM46: track 37.4 -> 36.6 mm
- net PWM30: track 37.4 -> 36.6 mm
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Other:
- outline, holes or cut-outs redrawn
- board text added: "12V"
- board text added: "48-Channel PWM Board v1.0 Designed by Linkun GAO"
- board text added: "5V"
- board text added: "A0"
- board text added: "A1"
- board text added: "A2"
- board text added: "A3"
- board text added: "A4"
- board text added: "A5"
- board text added: "D0"
- board text added: "D15"
- board text added: "D16"
- board text added: "D31"
- board text added: "D32"
- board text added: "D47"
- board text added: "SCL"
- board text added: "SDA"
- board text added: "~OE"

Commit message: v1.2 3v3 compatible
Parts:
- removed C1, C2: 47uF, Capacitor_THT:CP_Radial_D6.3mm_P2.50mm
- removed R21, R22: 1K, Resistor_SMD:R_0603_1608Metric
- added J6: Conn_01x02, Connector_PinSocket_2.54mm:PinSocket_1x02_P2.54mm_Vertical, F.Cu at (162.5, 36.0)
- R19, R20: value 10K -> 1K
- moved R20 97.5 mm to (151.0, 47.0), turned to 270 degrees
- moved R19 93.3 mm to (147.0, 47.0), turned to 270 degrees
- moved D49 1.00 mm to (147.0, 43.0)
- moved D50 1.00 mm to (151.0, 43.0)
Connections:
- C5 pad 1: +5V -> +3V3
- C6 pad 1: +5V -> +3V3
- C7 pad 1: +5V -> +3V3
- J5 pad 12: Net-(J5-Pad12) -> +3V3
- J5 pad 16: Net-(J5-Pad16) -> PSU_EN
- J5 pad 4: +5V -> Net-(J5-Pad4)
- J5 pad 7: Net-(J5-Pad7) -> GND
- JP1 pad 1: +5V -> +3V3
- JP10 pad 1: +5V -> +3V3
- JP11 pad 1: +5V -> +3V3
- JP12 pad 1: +5V -> +3V3
- JP13 pad 1: +5V -> +3V3
- JP14 pad 1: +5V -> +3V3
- JP15 pad 1: +5V -> +3V3
- JP16 pad 1: +5V -> +3V3
- JP17 pad 1: +5V -> +3V3
- JP18 pad 1: +5V -> +3V3
- JP2 pad 1: +5V -> +3V3
- JP3 pad 1: +5V -> +3V3
- JP4 pad 1: +5V -> +3V3
- JP5 pad 1: +5V -> +3V3
- JP6 pad 1: +5V -> +3V3
- JP7 pad 1: +5V -> +3V3
- JP8 pad 1: +5V -> +3V3
- JP9 pad 1: +5V -> +3V3
- R19 pad 1: +5V -> Net-(D49-Pad2)
- R19 pad 2: SDA -> +12V
- R20 pad 1: +5V -> Net-(D50-Pad2)
- R20 pad 2: SCL -> +3V3
- U1 pad 28: +5V -> +3V3
- U2 pad 28: +5V -> +3V3
- U3 pad 28: +5V -> +3V3
Routing:
- net +5V: track 295.1 -> 0.00 mm, vias 6 -> 0
- net +3V3: track 0.00 -> 257.4 mm, vias 0 -> 6
- net PSU_EN: track 0.00 -> 48.5 mm
- net +12V: track 610.5 -> 619.6 mm
- net SCL: track 209.9 -> 206.2 mm
- net SDA: track 206.1 -> 203.8 mm
- net /A35: track 58.2 -> 56.8 mm
- net /A15: track 58.4 -> 57.1 mm
- net /A25: track 58.3 -> 57.1 mm
Other:
- board text added: "3V3"
- board text added: "48-Channel PWM Board v1.2 Designed by Linkun GAO"
- board text added: "IC1"
- board text added: "IC2"
- board text added: "IC3"
- board text removed: "48-Channel PWM Board v1.0 Designed by Linkun GAO"
- board text removed: "5V"
