File: PWM-PCA9685.sch (KiCad schematic (older format))
At the start: 121 parts, among them J1 Conn_02x16_Top_Bottom, J2 Conn_02x16_Top_Bottom, J3 Conn_02x16_Top_Bottom, J4 Conn_02x20_Odd_Even, J5 Conn_02x12_Top_Bottom, Q1 SQJB00EP-T1_GE3, Q10 SQJB00EP-T1_GE3, Q11 SQJB00EP-T1_GE3, Q12 SQJB00EP-T1_GE3, Q13 SQJB00EP-T1_GE3, Q14 SQJB00EP-T1_GE3, Q15 SQJB00EP-T1_GE3, Q16 SQJB00EP-T1_GE3, Q17 SQJB00EP-T1_GE3, Q18 SQJB00EP-T1_GE3, Q19 SQJB00EP-T1_GE3, Q2 SQJB00EP-T1_GE3, Q20 SQJB00EP-T1_GE3, Q21 SQJB00EP-T1_GE3, Q22 SQJB00EP-T1_GE3, Q23 SQJB00EP-T1_GE3, Q24 SQJB00EP-T1_GE3, Q3 SQJB00EP-T1_GE3, Q4 SQJB00EP-T1_GE3, Q5 SQJB00EP-T1_GE3, Q6 SQJB00EP-T1_GE3, Q7 SQJB00EP-T1_GE3, Q8 SQJB00EP-T1_GE3, Q9 SQJB00EP-T1_GE3, U1 PCA9685PW, U2 PCA9685PW, U3 PCA9685PW

Commit message: updated
Parts:
- added C1, C2, C3, C4: 47uF, Capacitor_THT:CP_Radial_D6.3mm_P2.50mm, symbol Device:CP1_Small
- added D49, D50: LED, LED_SMD:LED_0603_1608Metric, symbol Device:LED
- added R21, R22: 1K, Resistor_SMD:R_0603_1608Metric, symbol Device:R_Small
- C5: renamed from C1; footprint Capacitor_SMD:C_0603_1608Metric -> Capacitor_SMD:C_1206_3216Metric
- C6: renamed from C2; footprint Capacitor_SMD:C_0603_1608Metric -> Capacitor_SMD:C_1206_3216Metric
- C7: renamed from C3; footprint Capacitor_SMD:C_0603_1608Metric -> Capacitor_SMD:C_1206_3216Metric
Connections:
- net +12V: now also C3.1, C4.1, R21.2
- net +5V: now also C1.1, C2.1, R22.2
- net GND: now also C1.2, C2.2, C3.2, C4.2, D49.1 (K), D50.1 (K); no longer U1.23 (~OE), U2.23 (~OE), U3.23 (~OE)
- net ~OE: now reaches J4.40 (Pin_40)
- net ~OE: now also U1.23 (~OE), U2.23 (~OE), U3.23 (~OE)
- new net: D49.2 (A), R21.1
- new net: D50.2 (A), R22.1
- no-connect marks 45 -> 44

Commit message: v1.2 3v3 compatible
Parts:
- removed C1, C2: 47uF, Capacitor_THT:CP_Radial_D6.3mm_P2.50mm, symbol Device:CP1_Small
- removed R19, R20: 10K, Resistor_SMD:R_0603_1608Metric, symbol Device:R_Small
- added J6: Conn_01x02, Connector_PinSocket_2.54mm:PinSocket_1x02_P2.54mm_Vertical, symbol Connector_Generic:Conn_01x02
- renumbered R21 to R19, R22 to R20
Connections:
- net GND: now also J5.7 (Pin_7), J6.2 (Pin_2)
- net +3V3: now reaches J5.12 (Pin_12)
- net +3V3: now also C5.1, C6.1, C7.1, JP1.1 (A), JP10.1 (A), JP11.1 (A), JP12.1 (A), JP13.1 (A), JP14.1 (A), JP15.1 (A), JP16.1 (A), JP17.1 (A), JP18.1 (A), JP2.1 (A), JP3.1 (A), JP4.1 (A), JP5.1 (A), JP6.1 (A), JP7.1 (A), JP8.1 (A), JP9.1 (A), R20.2, U1.28 (VDD), U2.28 (VDD), U3.28 (VDD)
- net PSU_EN: now reaches J5.16 (Pin_16)
- net PSU_EN: now also J6.1 (Pin_1)
- removed net +5V: C5.1, C6.1, C7.1, J5.4 (Pin_4), JP1.1 (A), JP10.1 (A), JP11.1 (A), JP12.1 (A), JP13.1 (A), JP14.1 (A), JP15.1 (A), JP16.1 (A), JP17.1 (A), JP18.1 (A), JP2.1 (A), JP3.1 (A), JP4.1 (A), JP5.1 (A), JP6.1 (A), JP7.1 (A), JP8.1 (A), JP9.1 (A), R20.2, U1.28 (VDD), U2.28 (VDD), U3.28 (VDD)
- no-connect marks 44 -> 42
